File: PCB/PCBMINI3.brd (EAGLE design)
At the start: 85 x 83.7 mm, 61 parts, among them IC101 TPS73533DRB, J1 DCJ0202, J6 HEADER 1X03, J7 BP_HEADERS_PWR_5V, U2 LM1084IS-5.0

Commit message: Add files via upload
Parts:
- moved LEDR1 3.81 mm to (7.62, 43.2)
- moved LEDR2 3.81 mm to (7.62, 35.6)
- moved LEDY1 3.81 mm to (7.62, 19.1)
- moved LEDY2 3.81 mm to (7.62, 26.7)
- moved LV3HP1 3.81 mm to (7.62, 53.3)
- moved LV3HP2 3.81 mm to (7.62, 66.0)
- moved R3 1.27 mm to (50.8, 19.1)
- turned C12 to 0 degrees
- turned C2 to 180 degrees
- turned R10 to 180 degrees
Routing:
- net +12V: track 164.1 -> 207.1 mm
- net P7.7: track 98.8 -> 63.3 mm
- net GND: track 500.3 -> 523.5 mm
- net P1.6_SPIMOSI_J2.15: track 120.6 -> 103.2 mm, vias 2 -> 3
- net +5V: track 311.7 -> 325.1 mm
- net P7.6: track 82.8 -> 70.5 mm
- net P6.5_I2CSCL_J1.9: track 104.6 -> 114.8 mm
- net N$7: track 19.6 -> 13.1 mm
- net XDSET_VCC: track 218.5 -> 224.4 mm
- net R2: track 37.0 -> 40.8 mm
- net Y1: track 16.0 -> 19.8 mm
- net N$1: track 16.9 -> 20.8 mm
- net R1: track 35.7 -> 39.3 mm
- net N$6: track 59.9 -> 57.6 mm
- net P5.2/XT2IN: track 45.5 -> 43.7 mm
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
Commit message: Add files via upload
Parts:
- removed C13, C9: 10u, eagle-ltspice:C0805
- removed R10: 365Ohms, eagle-ltspice:R0805
- removed TRANSR1, TRANSR2, TRANSY1, TRANSY2: STN2NF10, STN2NF10:SOT230P700X180-4N
- removed U2: LM1084IS-5.0, LM1084IS-5.0:TO254P1435X457-3N
- added 12TO5: TPS563200DDCR, TPS563200DDCR:SOT95P280X110-6N
- added C16, C21: 10u, eagle-ltspice:C0805
- added C17, C20, C24: 22u, eagle-ltspice:C0805
- added C18, C23: 0.1u, eagle-ltspice:C0805
- added L2: 3.3uH, Murata:0806
- added R11: 54.9k, eagle-ltspice:R0805
- added R12: 10k, eagle-ltspice:R0805
- added T1, T2, T3, T4: 2N7002-7-F, 2N7002-7-F:SOT103P240X110-3N
- R9: value 121Ohms -> 10k
- moved R9 136.6 mm to (-29.2, -73.7)
- moved LEDR1 62.7 mm to (0.00, -19.1), turned to 0 degrees
- moved LEDR2 54.6 mm to (7.62, -19.1), turned to 0 degrees
- moved LEDY2 48.2 mm to (22.9, -19.1), turned to 0 degrees
- moved LEDY1 38.9 mm to (15.2, -19.1), turned to 0 degrees
- moved LV3HP1 3.81 mm to (11.4, 53.3)
- moved LV3HP2 3.81 mm to (11.4, 66.0)
- moved R3 1.27 mm to (52.1, 19.1)
- turned C12 to 180 degrees
- turned C2 to 0 degrees
Connections:
- removed net R1: LEDR1.1, TRANSR1.2, TRANSR1.4
- removed net R2: LEDR2.1, TRANSR2.2, TRANSR2.4
- new net N$12: 12TO5.6, C23.1
- new net N$13: 12TO5.4, R11.1, R9.2
- new net N$4: 12TO5.5, R12.2
- new net N$5: LEDR1.1, T1.3
- new net N$8: C17.1, C20.1, C24.1, L2.1, R11.2
- new net N$9: LEDR2.1, T2.3
- net +12V: now also 12TO5.3, C16.1, C18.1, C21.1, R12.1; no longer C9.1, U2.3
- net +5V: no longer C13.2, R9.2, U2.4
- net GND: now also 12TO5.1, C16.2, C17.2, C18.2, C20.2, C21.2, C24.2, R9.1, T1.2, T2.2, T3.2, T4.2; no longer C13.1, C9.2, R10.1, TRANSR1.3, TRANSR2.3, TRANSY1.3, TRANSY2.3
- net N$1: now also T4.3; no longer TRANSY2.2, TRANSY2.4
- net N$7: now also 12TO5.2, C23.2, L2.2; no longer R10.2, R9.1, U2.1
- net P7.4: now also T1.1; no longer TRANSR1.1
- net P7.5: now also T2.1; no longer TRANSR2.1
- net P7.6: now also T3.1; no longer TRANSY1.1
- net P7.7: now also T4.1; no longer TRANSY2.1
- net Y1: now also T3.3; no longer TRANSY1.2, TRANSY1.4
Routing:
- net +12V: track 207.1 -> 134.8 mm
- net GND: track 523.5 -> 462.8 mm, vias 14 -> 12
- net R2: track 40.8 -> 0.00 mm
- net R1: track 39.3 -> 0.00 mm
- net P7.7: track 63.3 -> 98.7 mm
- net +5V: track 325.1 -> 299.9 mm
- net N$1: track 20.8 -> 0.00 mm
- net Y1: track 19.8 -> 0.00 mm
- net P1.6_SPIMOSI_J2.15: track 103.2 -> 120.6 mm, vias 3 -> 2
- net N$7: track 13.1 -> 0.00 mm
- net P7.6: track 70.5 -> 82.7 mm
- net P6.5_I2CSCL_J1.9: track 114.8 -> 104.6 mm
- net XDSET_VCC: track 224.4 -> 218.5 mm
- net N$6: track 57.6 -> 59.9 mm
- net P5.2/XT2IN: track 43.7 -> 45.5 mm
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