File: PCB/PCBMINI3.sch (EAGLE design)
At the start: 61 parts, among them IC101 TPS73533DRB, J1 DCJ0202, J6 HEADER 1X03, J7 BP_HEADERS_PWR_5V, U2 LM1084IS-5.0

Commit message: Add files via upload
Parts:
- removed C13, C9: 10u, eagle-ltspice:C
- removed R10: 365Ohms, eagle-ltspice:R
- removed TRANSR1, TRANSR2, TRANSY1, TRANSY2: STN2NF10, STN2NF10:STN2NF10
- removed U2: LM1084IS-5.0, LM1084IS-5.0:LM1084IS-5.0
- added 12TO5: TPS563200DDCR, TPS563200DDCR:TPS563200DDCR
- added C16, C21: 10u, eagle-ltspice:C
- added C17, C20, C24: 22u, eagle-ltspice:C
- added C18, C23: 0.1u, eagle-ltspice:C
- added L2: 3.3uH, Murata:LQM2MP_G0
- added R11: 54.9k, eagle-ltspice:R
- added R12: 10k, eagle-ltspice:R
- added T1, T2, T3, T4: 2N7002-7-F, 2N7002-7-F:2N7002-7-F
- R9: value 121Ohms -> 10k
Connections:
- removed net R1: LEDR1.1, TRANSR1.D@1, TRANSR1.D@2
- removed net R2: LEDR2.1, TRANSR2.D@1, TRANSR2.D@2
- new net N$12: 12TO5.VBST, C23.1
- new net N$13: 12TO5.VFB, R11.1, R9.2
- new net N$4: 12TO5.EN, R12.2
- new net N$5: LEDR1.1, T1.D
- new net N$8: C17.1, C20.1, C24.1, L2.1, R11.2
- new net N$9: LEDR2.1, T2.D
- net +12V: now also 12TO5.VIN, C16.1, C18.1, C21.1, R12.1; no longer C9.1, U2.IN
- net +5V: no longer C13.2, R9.2, U2.VOUT
- net GND: now also 12TO5.GND, C16.2, C17.2, C18.2, C20.2, C21.2, C24.2, R9.1, T1.S, T2.S, T3.S, T4.S; no longer C13.1, C9.2, R10.1, TRANSR1.S, TRANSR2.S, TRANSY1.S, TRANSY2.S
- net N$1: now also T4.D; no longer TRANSY2.D@1, TRANSY2.D@2
- net N$7: now also 12TO5.SW, C23.2, L2.2; no longer R10.2, R9.1, U2.ADJ/GND
- net P7.4: now also T1.G; no longer TRANSR1.G
- net P7.5: now also T2.G; no longer TRANSR2.G
- net P7.6: now also T3.G; no longer TRANSY1.G
- net P7.7: now also T4.G; no longer TRANSY2.G
- net Y1: now also T3.D; no longer TRANSY1.D@1, TRANSY1.D@2
Other:
- moved on the sheet: LEDR1, LEDR2, LEDY1, LEDY2, R9
